File: Schemat/Schemat.kicad_sch (KiCad schematic)
At the start: 47 parts, among them J1 Złącze mikrokontrolera, J2 Screw_Terminal_01x02, J3 Screw_Terminal_01x02, J4 Screw_Terminal_01x02, J5 Screw_Terminal_01x02, J6 Screw_Terminal_01x02, J7 Zasilanie 5V, K1 SRD, K2 SRD, K3 SRD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

Commit message: Sterowanie żarówką przy pomocy przycisku
Parts:
- removed D1, D10, D4, D6, D8: 1N4007, symbol Device:D
- removed D2, D3, D5, D7, D9: LED, symbol Device:LED
- removed J1: Złącze mikrokontrolera, symbol Connector:Conn_01x05_Male
- removed J2, J3, J4, J5, J6: Screw_Terminal_01x02, symbol Connector:Screw_Terminal_01x02
- removed J7: Zasilanie 5V, symbol Connector:Screw_Terminal_01x02
- removed K1, K2, K3, K4, K5: SRD, Relay_THT:Relay_SPDT_Finder_36.11, symbol Relay:FINDER-36.11
- removed Q2, Q3, Q4, Q5: BC107, Package_TO_SOT_SMD:SOT-23, symbol Transistor_BJT:BC849
- removed R10, R13, R4, R7: 1k, symbol Device:R
- removed R11, R12, R14, R15, R5, R6, R8, R9: 10k, symbol Device:R
- removed U2, U3, U4: LTV 814, Package_SO:SOP-4_4.4x2.6mm_P1.27mm, symbol Isolator:ACPL-214-500E
- removed U5: LTV 814, symbol Isolator:ACPL-214-500E
- added C1: 100n, symbol Device:C
- added SW1: Switch, symbol Switch:SW_DIP_x01
- Q1: value BC107 -> 2N3055
- R1: value 1k -> 120
- R2: value 10k -> 2,7k
- R3: value 10k -> Light bulb 12V 5W
Connections:
- net GND: now also U1.3, C1.2, SW1.2
- net at R2.2, U1.4: now also Q1.1 (B)
- net at R3.2: now also Q1.3 (C)
- net +5V renamed +12V
- net uC_1 renamed RF0
- new net RF1: C1.1, SW1.1
Other:
- moved on the sheet: Q1, R1, R2, U1
